File: DSPicPiHat/_autosave-DSPicPiHat.kicad_pcb (KiCad board)
At the start: 2 copper layers, 67 x 66.5 mm, 89 parts, among them J10 Nice!View, J4 Conn_PIC_ICSP_ICD, J5 USB_C_Receptacle_USB2.0, J6 PowerInput, J7 GenericSPIconn, J8 RasPiHeaders, J9 GeneralSPIDisplay, SW1 POWER_Select, SW2 SW_DIP_x08, U1 DSPIC33CH512MP508T-I_PT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

Commit message: Connected all the coil driver connectors. Added more footprints.
Parts:
- added L1: 10 mA <1o, Inductor_SMD:L_0805_2012Metric, F.Cu at (86.8, 117.0)
- C19, C22: footprint Capacitor_SMD:C_1206_3216Metric -> Capacitor_SMD:C_0805_2012Metric
- C21: footprint Capacitor_SMD:CP_Elec_4x5.8 -> Capacitor_SMD:C_0805_2012Metric
- moved C4 157.5 mm to (97.6, 128.6)
- moved C8 144.0 mm to (114.2, 128.2), turned to 90 degrees
- moved C11 131.7 mm to (98.0, 120.2)
- moved U1 129.8 mm to (99.5, 108.5)
- moved C2 129.6 mm to (78.4, 128.6)
- moved C10 120.3 mm to (89.8, 109.2), turned to 180 degrees
- moved C12 117.1 mm to (89.2, 115.2), turned to -90 degrees
- moved D3 6.26 mm to (116.2, 122.2)
- moved D2 3.32 mm to (99.4, 125.8)
- moved D1 3.16 mm to (80.0, 125.8)
- moved R5 0.10 mm to (114.1, 124.4)
Connections:
- U1 pad 15: EXT_ADC_X_03 -> EXT_Y_PWM_00
- U1 pad 28: unconnected-(U1-Pad28) -> EXT_Y_PWM_01
- U1 pad 29: unconnected-(U1-Pad29) -> EXT_ADC_Y_00
- U1 pad 3: EXT_Y_PWM_00 -> EXT_X_PWM_01
- U1 pad 30: unconnected-(U1-Pad30) -> EXT_ADC_Y_01
- U1 pad 33: unconnected-(U1-Pad33) -> EXT_ADC_Y_02
- U1 pad 40: unconnected-(U1-Pad40) -> EXT_ADC_Y_03
- U1 pad 41: EXT_ADC_Y_00 -> EXT_Z_PWM_00
- U1 pad 43: EXT_ADC_Y_01 -> EXT_Z_PWM_01
- U1 pad 45: EXT_ADC_Y_02 -> EXT_ADC_Z_00
- U1 pad 46: EXT_ADC_Y_03 -> EXT_ADC_Z_01
- U1 pad 47: unconnected-(U1-Pad47) -> EXT_ADC_Z_02
- U1 pad 5: EXT_Z_PWM_00 -> EXT_ADC_X_00
- U1 pad 52: unconnected-(U1-Pad52) -> EXT_ADC_Z_03
- U1 pad 6: EXT_ADC_X_00 -> EXT_ADC_X_01
- U1 pad 63: EXT_ADC_Z_00 -> unconnected-(U1-Pad63)
- U1 pad 65: EXT_ADC_Z_01 -> unconnected-(U1-Pad65)
- U1 pad 66: EXT_ADC_Z_02 -> unconnected-(U1-Pad66)
- U1 pad 67: EXT_ADC_Z_03 -> unconnected-(U1-Pad67)
- U1 pad 7: EXT_ADC_X_01 -> EXT_ADC_X_02
- U1 pad 72: EXT_Z_PWM_01 -> unconnected-(U1-Pad72)
- U1 pad 73: EXT_Y_PWM_01 -> unconnected-(U1-Pad73)
- U1 pad 74: EXT_X_PWM_01 -> unconnected-(U1-Pad74)
- U1 pad 8: EXT_ADC_X_02 -> EXT_ADC_X_03
Routing:
- net EXT_X_PWM_00: track 12.5 -> 52.1 mm
- net EXT_X_PWM_01: track 12.8 -> 51.2 mm
- net EXT_ADC_X_00: track 10.0 -> 46.9 mm
- net EXT_ADC_X_01: track 7.81 -> 44.1 mm
- net EXT_ADC_X_02: track 9.11 -> 44.2 mm, vias 3 -> 2
- net EXT_ADC_X_03: track 11.1 -> 45.2 mm
- net EXT_ADC_Z_03: track 15.8 -> 41.3 mm
- net EXT_Y_PWM_01: track 7.91 -> 33.3 mm
- net EXT_Y_PWM_00: track 7.88 -> 33.2 mm
- net EXT_ADC_Y_03: track 12.7 -> 37.3 mm
- net U1CTS: track 0.00 -> 23.9 mm
- net U1RX: track 0.00 -> 21.6 mm, vias 0 -> 2
- net EXT_ADC_Y_02: track 10.4 -> 31.8 mm, vias 1 -> 2
- net EXT_ADC_Y_00: track 9.74 -> 31.0 mm
- net U1RTS: track 0.00 -> 20.9 mm
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